File: hardware/video_and_power.brd (EAGLE design)
At the start: 151.4 x 117.5 mm, 37 parts, among them IC1 74HCT574N, IC2 74HCT574N, IC3 74HCT574N, IC4 74HCT04N, IC5 7432N, IC7 7805T, J2 POWER_JACKSLT, X1 736880-49

Commit message: PCB update
Parts:
- removed B1: DBDB101G, rectifier:DB
- added Q4: (no value), transistor-power:SO-08
- added R25: 1k, rcl:R0603
Connections:
- removed net N$12: B1.AC2, J2.GND@1, J2.GND@2
- removed net N$14: B1.+, C1.1, C5.+, IC7.1
- new net 9V: C1.1, C5.+, IC7.1, Q4.1, Q4.2, Q4.3
- new net N$52: F2.2, Q4.5, Q4.6, Q4.7, Q4.8
- net GND: now also J2.GND@1, J2.GND@2, R25.1; no longer B1.-
- net N$3: now also Q4.4, R25.2; no longer B1.AC1, F2.2
Routing:
- net N$12: track 49.0 -> 0.00 mm
- net 9V: track 0.00 -> 37.5 mm
- net N$14: track 33.7 -> 0.00 mm
- net GND: track 34.3 -> 42.6 mm
- net N$3: track 3.99 -> 2.63 mm
- added copper zone on layer 16, net 9V
- added copper zone on layer 16, net N$52
Changed lines of the file:
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@@
 <?xml version="1.0" encoding="utf-8"?>
 <!DOCTYPE eagle SYSTEM "eagle.dtd">
-<eagle version="7.2.0">
+<eagle version="7.7.0">
 <drawing>
 <settings>
@@
 <layer number="154" name="FabDoc2" color="7" fill="1" visible="no" active="yes"/>
 <layer number="155" name="FabDoc3" color="7" fill="1" visible="no" active="yes"/>
+<layer number="156" name="gesam-Maß" color="1" fill="7" visible="no" active="no"/>
+<layer number="157" name="FaceMchng" color="3" fill="1" visible="no" active="no"/>
+<layer number="158" name="FaceMMeas" color="3" fill="1" visible="no" active="no"/>
+<layer number="159" name="Geh-Bear2" color="1" fill="7" visible="no" active="no"/>
+<layer number="160" name="Topologie" color="9" fill="1" visible="no" active="no"/>
+<layer number="161" name="tomplace2" color="7" fill="1" visible="no" active="no"/>
 <layer number="191" name="mNets" color="7" fill="1" visible="no" active="yes"/>
 <layer number="192" name="mBusses" color="7" fill="1" visible="no" active="yes"/>
@@
 <layer number="250" name="Descript" color="3" fill="1" visible="no" active="no"/>
 <layer number="251" name="SMDround" color="12" fill="11" visible="no" active="no"/>
+<layer number="252" name="BR-BS" color="7" fill="1" visible="no" active="no"/>
+<layer number="253" name="BR-LS" color="7" fill="1" visible="no" active="no"/>
 <layer number="254" name="cooling" color="7" fill="1" visible="no" active="yes"/>
 <layer number="255" name="HELP" color="7" fill="1" visible="no" active="yes"/>
@@
 <element name="R4" library="rcl" package="R0805" value="" x="137.4775" y="99.695" rot="MR180"/>
 <element name="C4" library="rcl" package="C0603" value="" x="133.985" y="96.52" rot="MR270"/>
-<element name="B1" library="rectifier" package="DB" value="DBDB101G" x="26.035" y="62.23"/>
 <element name="C5" library="rcl" package="E5-10,5" value="" x="26.035" y="51.435"/>
 <element name="C6" library="rcl" package="E5-10,5" value="" x="45.72" y="38.1" rot="R270"/>
@@
 <element name="JP1" library="pinhead" package="1X02" value="" x="28.575" y="98.1075" rot="R270"/>
 <element name="IC5" library="74xx-us" package="DIL14" value="7432N" x="108.585" y="30.1625" rot="R270"/>
+<element name="Q4" library="transistor-power" package="SO-08" value="" x="26.0858" y="61.595" rot="MR90"/>
+<element name="R25" library="rcl" package="R0603" value="1k" x="20.0025" y="63.5" rot="MR180"/>
 </elements>
 <signals>
@@
 </signal>
 <signal name="GND">
-<polygon width="0.4064" layer="16" isolate="0.6096" thermals="no">
+<polygon width="0.4064" layer="16" isolate="0.6096" thermals="no" rank="2">
 <vertex x="17.78" y="117.475"/>
 <vertex x="17.78" y="43.18"/>
@@
 <via x="126.365" y="80.645" extent="1-16" drill="0.6" diameter="1.4224" shape="octagon"/>
 <wire x1="126.365" y1="66.675" x2="126.365" y2="80.645" width="0.6096" layer="1"/>
-<contactref element="B1" pad="-"/>
 <contactref element="C1" pad="2"/>
 <contactref element="C2" pad="2"/>
@@
 <via x="67.945" y="110.8075" extent="1-16" drill="0.6" diameter="1.4224" shape="octagon"/>
 <via x="67.945" y="105.7275" extent="1-16" drill="0.6" diameter="1.4224" shape="octagon"/>
-<via x="33.655" y="64.77" extent="1-16" drill="0.6" diameter="1.4224" shape="octagon"/>
-<via x="38.735" y="64.77" extent="1-16" drill="0.6" diameter="1.4224" shape="octagon"/>
-<wire x1="38.735" y1="64.77" x2="33.655" y2="64.77" width="0.6096" layer="1"/>
+<via x="33.655" y="65.405" extent="1-16" drill="0.6" diameter="1.4224" shape="octagon"/>
+<via x="38.735" y="65.405" extent="1-16" drill="0.6" diameter="1.4224" shape="octagon"/>
+<wire x1="38.735" y1="65.405" x2="33.655" y2="65.405" width="0.6096" layer="1"/>
 <wire x1="67.945" y1="105.7275" x2="67.945" y2="110.8075" width="0.6096" layer="1"/>
 <via x="81.915" y="110.8075" extent="1-16" drill="0.6" diameter="1.4224" shape="octagon"/>
@@
 <contactref element="IC5" pad="5"/>
 <contactref element="IC5" pad="10"/>
+<contactref element="R25" pad="1"/>
+<contactref element="J2" pad="GND@1"/>
+<contactref element="J2" pad="GND@2"/>
+<wire x1="28.5731" y1="109.975" x2="23.5604" y2="109.975" width="1.27" layer="16"/>
+<wire x1="23.5604" y1="109.975" x2="23.5731" y2="106.675" width="1.27" layer="16"/>
 </signal>
 <signal name="D0">
@@
 <wire x1="133.985" y1="99.695" x2="136.5275" y2="99.695" width="0.6096" layer="16"/>
 </signal>
-<signal name="N$12">
-<contactref element="J2" pad="GND@1"/>
-<contactref element="J2" pad="GND@2"/>
-<contactref element="B1" pad="AC2"/>
-<wire x1="23.5731" y1="106.675" x2="23.5604" y2="66.1054" width="1.27" layer="16"/>
-<wire x1="23.5604" y1="66.1054" x2="23.495" y2="66.04" width="1.27" layer="16"/>
-<wire x1="28.5731" y1="109.975" x2="23.5604" y2="109.975" width="1.27" layer="16"/>
-<wire x1="23.5604" y1="109.975" x2="23.5731" y2="106.675" width="1.27" layer="16"/>
-</signal>
-<signal name="N$3">
-<contactref element="B1" pad="AC1"/>
-<contactref element="F2" pad="2"/>
-<wire x1="28.575" y1="66.04" x2="28.575" y2="70.0278" width="1.27" layer="16"/>
-</signal>
-<signal name="N$14">
-<contactref element="B1" pad="+"/>
-<contactref element="IC7" pad="1"/>
-<wire x1="36.195" y1="35.56" x2="32.385" y2="35.56" width="1.27" layer="16"/>
-<wire x1="32.385" y1="35.56" x2="29.21" y2="38.735" width="1.27" layer="16"/>
-<contactref element="C1" pad="1"/>
-<wire x1="36.195" y1="35.56" x2="39.5575" y2="35.56" width="1.27" layer="16"/>
-<contactref element="C5" pad="+"/>
-<wire x1="23.495" y1="58.42" x2="23.495" y2="51.435" width="1.27" layer="16"/>
-<wire x1="29.21" y1="38.735" x2="29.21" y2="45.72" width="1.27" layer="16"/>
-<wire x1="29.21" y1="45.72" x2="23.495" y2="51.435" width="1.27" layer="16"/>
-</signal>
 <signal name="N$8">
 <contactref element="J2" pad="PWR"/>
@@
 <wire x1="28.575" y1="96.8375" x2="28.575" y2="92.5322" width="1.524" layer="16"/>
 </signal>
+<signal name="9V">
+<contactref element="Q4" pad="1"/>
+<contactref element="Q4" pad="3"/>
+<contactref element="Q4" pad="2"/>
+<contactref element="IC7" pad="1"/>
+<contactref element="C1" pad="1"/>
+<contactref element="C5" pad="+"/>
+<wire x1="36.195" y1="35.56" x2="32.385" y2="35.56" width="1.27" layer="16"/>
+<wire x1="32.385" y1="35.56" x2="29.21" y2="38.735" width="1.27" layer="16"/>
+<wire x1="36.195" y1="35.56" x2="39.5575" y2="35.56" width="1.27" layer="16"/>
+<wire x1="29.21" y1="38.735" x2="29.21" y2="45.72" width="1.27" layer="16"/>
+<wire x1="29.21" y1="45.72" x2="23.495" y2="51.435" width="1.27" layer="16"/>
+<wire x1="23.495" y1="51.435" x2="23.495" y2="59.6808" width="0.6096" layer="16"/>
+<wire x1="23.495" y1="59.6808" x2="23.4858" y2="59.69" width="0.6096" layer="16"/>
+<wire x1="23.4858" y1="59.69" x2="23.4858" y2="60.96" width="0.6096" layer="16"/>
+<wire x1="23.4858" y1="60.96" x2="23.4858" y2="62.23" width="0.6096" layer="16"/>
+<polygon width="0.6096" layer="16" isolate="0.4064" thermals="no">
+<vertex x="24.765" y="50.165"/>
+<vertex x="22.225" y="50.165"/>
+<vertex x="22.225" y="62.2935"/>
+<vertex x="24.765" y="62.2935"/>
+</polygon>
+</signal>
+<signal name="N$52">
+<contactref element="Q4" pad="8"/>
+<contactref element="Q4" pad="6"/>
+<contactref element="Q4" pad="5"/>
+<contactref element="Q4" pad="7"/>
+<contactref element="F2" pad="2"/>
+<polygon width="0.6096" layer="16" isolate="0.3048" thermals="no">
+<vertex x="26.035" y="71.12"/>
+<vertex x="26.035" y="59.69"/>
+<vertex x="31.115" y="59.69"/>
+<vertex x="31.115" y="71.12"/>
+</polygon>
+</signal>
+<signal name="N$3">
+<contactref element="Q4" pad="4"/>
+<contactref element="R25" pad="2"/>
+<wire x1="23.4858" y1="63.5" x2="20.8525" y2="63.5" width="0.6096" layer="16"/>
+</signal>
 </signals>
